Commit message: feat: init LiDar not working

File: src/description/robot.urdf.xacro (robot description, xacro)
@@ -2,5 +2,7 @@
 <robot xmlns:xacro="http://www.ros.org/wiki/xacro"  name="robot">
     <xacro:include filename="robot_core.xacro" />
-    <!-- Plug in for gazebo control -->
+    <!-- File for gazebo control -->
     <xacro:include filename="gazebo_control.xacro" />
+    <!-- File for lidar control -->
+    <xacro:include filename="lidar.xacro" />
 </robot>

File: src/description/robot_core.xacro (robot description, xacro)
@@ -13,4 +13,7 @@
     <material name="black">
         <color rgba="0 0 0 1"/>
+    </material>
+    <material name="red">
+        <color rgba="1 0 0 1"/>
     </material>
     <!-- BASE LINK -->
