Commit message: fix: correctly closed xml tag

File: src/description/lidar.xacro (robot description, xacro)
@@ -22,5 +22,5 @@
         <xacro:inertial_cylinder mass="0.1" length="0.4" radius="0.05">
             <origin xyz="0 0 0" rpy="0 0 0"/>
-        </inertial>
+        </xacro:inertial_cylinder>
     </link>
 </robot>

Commit message: feat: add lidar to gazebo. Fixes #1

File: src/description/lidar.xacro (robot description, xacro)
@@ -24,3 +24,40 @@
         </xacro:inertial_cylinder>
     </link>
+    <!-- Add a gazebo tag to simulate the LiDar -->
+    <gazebo reference="laser_frame">
+        <!-- Set the color of the LiDar. The color for the link sets color in rviz, not Gazebo -->
+        <material>Gazebo/Red</material>
+        <!-- Ray sensor is a scanning LiDar -->
+        <sensor name="laser" type="ray">
+            <!-- Origin of the sensor is at the center of the link -->
+            <pose> 0 0 0 0 0 0 </pose>
+            <visualize>true</visualize>
+            <!-- Update 10 times / second -->
+            <update_rate>10</update_rate>
+            <!-- Specify paramters for the virtual sensor -->
+            <ray>
+                <scan>
+                    <horizontal>
+                        <samples>360</samples>
+                        <min_angle>-3.14</min_angle>
+                        <max_angle>3.14</max_angle>
+                    </horizontal>
+                </scan>
+                <range>
+                    <min>0.3</min>
+                    <max>12</max>
+                </range>
+            </ray>
+            <!-- Plug in to publish the gazebo ray sensor to ROS topics -->
+            <plugin name="laser_controller" filename="libgazebo_ros_ray_sensor.so">
+                <!-- What topic to publish onto (publish to scan) -->
+                <ros>
+                    <argument>~/out:=scan</argument>
+                </ros>
+                <output_type>sensor_msgs/LaserScan</output_type>
+                <!-- What frame ID to put in the laser scan message -->
+                <frame_name>laser_frame</frame_name>
+            </plugin>
+        </sensor>
+    </gazebo>
 </robot>
