Commit message: feat: add base_footprint joint

File: src/description/robot_core.xacro (robot description, xacro)
@@ -20,4 +20,10 @@
     <link name="base_link">
     </link>
+    <!-- BASE FOOTPRINT LINK -->
+    <joint name="base_footprint_joint" type="fixed">
+        <parent link="base_link"/>
+        <child link="base_footprint"/>
+        <origin xyz="0 0 0" rpy="0 0 0"/>
+    </joint>
     <!-- CHASSIS LINK -->
     <joint name="chassis_joint" type="fixed">

Commit message: slam_toolbox

File: src/description/robot_core.xacro (robot description, xacro)
@@ -26,4 +26,5 @@
         <origin xyz="0 0 0" rpy="0 0 0"/>
     </joint>
+    <link name="base_footprint"></link>
     <!-- CHASSIS LINK -->
     <joint name="chassis_joint" type="fixed">
